File: hw/shopie-hw/SnP.kicad_sch (KiCad schematic)
At the start: 20 parts, among them U5 HAKRC_Blehli32_ESC40A, U9 LTC2943

Commit message: Fix most ERC Errors and Connect hierarchical labels across schematic pages
- Connected missing net labels across MCU, Sensors, and Power pages
- Final ERC check passed with no errors or warnings for all labels
Connections:
- net BMP388_EN renamed BMP388_CS
- net ICM_EXTI renamed ICM20948_EXTI
Other:
- moved on the sheet: U5

Commit message: Fix remaining schematic ERC issues
- Resolved all remaining ERC errors across schematic sheets
- All power input pins are driven by valid power sources
Parts:
- gave numbers to parts that had none: 14
Changed lines of the file:
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@@
 	)
 	(junction
-		(at 158.75 49.53)
-		(diameter 0)
-		(color 0 0 0 0)
-	)
-	(junction
 		(at 264.16 87.63)
 		(diameter 0)
@@
 	)
 	(junction
+		(at 154.94 49.53)
+		(diameter 0)
+		(color 0 0 0 0)
+	)
+	(junction
 		(at 260.35 41.91)
 		(diameter 0)
@@
 	(wire
 		(pts
+			(xy 154.94 49.53) (xy 154.94 53.34)
+		)
+		(stroke
+			(width 0)
+			(type default)
+		)
+	)
+	(wire
+		(pts
 			(xy 30.48 102.87) (xy 33.02 102.87)
 		)
@@
 	(wire
 		(pts
+			(xy 154.94 49.53) (xy 158.75 49.53)
+		)
+		(stroke
+			(width 0)
+			(type default)
+		)
+	)
+	(wire
+		(pts
 			(xy 207.01 87.63) (xy 207.01 92.71)
 		)
@@
 	(wire
 		(pts
-			(xy 149.86 49.53) (xy 158.75 49.53)
+			(xy 149.86 49.53) (xy 154.94 49.53)
 		)
 		(stroke
@@
 	(wire
 		(pts
-			(xy 137.16 49.53) (xy 149.86 49.53)
-		)
-		(stroke
-			(width 0)
-			(type default)
-		)
-	)
-	(wire
-		(pts
 			(xy 247.65 44.45) (xy 247.65 52.07)
 		)
@@
 	(wire
 		(pts
-			(xy 158.75 53.34) (xy 158.75 49.53)
-		)
-		(stroke
-			(width 0)
-			(type default)
-		)
-	)
-	(wire
-		(pts
 			(xy 149.86 39.37) (xy 149.86 35.56)
 		)
@@
 	(wire
 		(pts
+			(xy 137.16 49.53) (xy 149.86 49.53)
+		)
+		(stroke
+			(width 0)
+			(type default)
+		)
+	)
+	(wire
+		(pts
 			(xy 200.66 39.37) (xy 200.66 49.53)
 		)
@@
 		(on_board yes)
 		(dnp no)
-		(property "Reference" "U?"
+		(property "Reference" "U302"
 			(at 127.254 29.464 0)
 			(effects
@@
 			(project "shopie-hw"
 				(path "/e9514a67-47f8-4b41-a728-bdf26e012bf7/d28d3f47-b0c1-4fbb-bdab-a8b85a0388d0"
-					(reference "U?")
+					(reference "U302")
 					(unit 1)
 				)
@@
 	(symbol
 		(lib_id "power:GND")
-		(at 158.75 53.34 0)
+		(at 154.94 53.34 0)
 		(unit 1)
 		(exclude_from_sim no)
@@
 		(dnp no)
 		(property "Reference" "#PWR0108"
-			(at 158.75 59.69 0)
+			(at 154.94 59.69 0)
 			(effects
 				(font
@@
 		)
 		(property "Value" "GND"
-			(at 158.75 57.404 0)
+			(at 154.94 57.404 0)
 			(effects
 				(font
@@
 		)
 		(property "Footprint" ""
-			(at 158.75 53.34 0)
+			(at 154.94 53.34 0)
 			(effects
 				(font
@@
 		)
 		(property "Datasheet" ""
-			(at 158.75 53.34 0)
+			(at 154.94 53.34 0)
 			(effects
 				(font
@@
 		)
 		(property "Description" "Power symbol creates a global label with name \"GND\" , ground"
-			(at 158.75 53.34 0)
+			(at 154.94 53.34 0)
 			(effects
 				(font
@@
 		(on_board yes)
 		(dnp no)
-		(property "Reference" "C?"
+		(property "Reference" "C307"
 			(at 261.62 46.228 0)
 			(effects
@@
 			(project "shopie-hw"
 				(path "/e9514a67-47f8-4b41-a728-bdf26e012bf7/d28d3f47-b0c1-4fbb-bdab-a8b85a0388d0"
-					(reference "C?")
+					(reference "C307")
 					(unit 1)
 				)
@@
 		(on_board yes)
 		(dnp no)
-		(property "Reference" "C?"
+		(property "Reference" "C301"
 			(at 40.386 27.94 90)
 			(effects
@@
 			(project "shopie-hw"
 				(path "/e9514a67-47f8-4b41-a728-bdf26e012bf7/d28d3f47-b0c1-4fbb-bdab-a8b85a0388d0"
-					(reference "C?")
+					(reference "C301")
 					(unit 1)
 				)
@@
 		(on_board yes)
 		(dnp no)
-		(property "Reference" "R?"
+		(property "Reference" "R302"
 			(at 199.39 49.53 0)
 			(effects
@@
 			(project "shopie-hw"
 				(path "/e9514a67-47f8-4b41-a728-bdf26e012bf7/d28d3f47-b0c1-4fbb-bdab-a8b85a0388d0"
-					(reference "R?")
+					(reference "R302")
 					(unit 1)
 				)
@@
 		(on_board yes)
 		(dnp no)
-		(property "Reference" "R?"
+		(property "Reference" "R301"
 			(at 190.5 50.8 0)
 			(effects
@@
 			(project "shopie-hw"
 				(path "/e9514a67-47f8-4b41-a728-bdf26e012bf7/d28d3f47-b0c1-4fbb-bdab-a8b85a0388d0"
-					(reference "R?")
+					(reference "R301")
 					(unit 1)
 				)
@@
 		(on_board yes)
 		(dnp no)
-		(property "Reference" "C?"
+		(property "Reference" "C303"
 			(at 75.946 55.88 90)
 			(effects
@@
 			(project "shopie-hw"
 				(path "/e9514a67-47f8-4b41-a728-bdf26e012bf7/d28d3f47-b0c1-4fbb-bdab-a8b85a0388d0"
-					(reference "C?")
+					(reference "C303")
 					(unit 1)
 				)
@@
 		(on_board yes)
 		(dnp no)
-		(property "Reference" "C?"
+		(property "Reference" "C308"
 			(at 264.16 28.448 0)
 			(effects
@@
 			(project "shopie-hw"
 				(path "/e9514a67-47f8-4b41-a728-bdf26e012bf7/d28d3f47-b0c1-4fbb-bdab-a8b85a0388d0"
-					(reference "C?")
+					(reference "C308")
 					(unit 1)
 				)
@@
 		(on_board yes)
 		(dnp no)
-		(property "Reference" "C?"
+		(property "Reference" "C302"
 			(at 66.294 27.94 90)
 			(effects
@@
 			(project "shopie-hw"
 				(path "/e9514a67-47f8-4b41-a728-bdf26e012bf7/d28d3f47-b0c1-4fbb-bdab-a8b85a0388d0"
-					(reference "C?")
+					(reference "C302")
 					(unit 1)
 				)
@@
 		(on_board yes)
 		(dnp no)
-		(property "Reference" "U?"
+		(property "Reference" "U303"
 			(at 238.252 25.4 0)
 			(effects
@@
 			(project "shopie-hw"
 				(path "/e9514a67-47f8-4b41-a728-bdf26e012bf7/d28d3f47-b0c1-4fbb-bdab-a8b85a0388d0"
-					(reference "U?")
+					(reference "U303")
 					(unit 1)
 				)
@@
 		(on_board yes)
 		(dnp no)
-		(property "Reference" "C?"
+		(property "Reference" "C304"
 			(at 151.13 41.148 0)
 			(effects
@@
 			(project "shopie-hw"
 				(path "/e9514a67-47f8-4b41-a728-bdf26e012bf7/d28d3f47-b0c1-4fbb-bdab-a8b85a0388d0"
-					(reference "C?")
+					(reference "C304")
 					(unit 1)
 				)
@@
 		(on_board yes)
 		(dnp no)
-		(property "Reference" "R?"
+		(property "Reference" "R303"
 			(at 204.47 53.34 0)
 			(effects
@@
 			(project "shopie-hw"
 				(path "/e9514a67-47f8-4b41-a728-bdf26e012bf7/d28d3f47-b0c1-4fbb-bdab-a8b85a0388d0"
-					(reference "R?")
+					(reference "R303")
 					(unit 1)
 				)
@@
 		(on_board yes)
 		(dnp no)
-		(property "Reference" "C?"
+		(property "Reference" "C306"
 			(at 177.8 34.798 0)
 			(effects
@@
 			(project "shopie-hw"
 				(path "/e9514a67-47f8-4b41-a728-bdf26e012bf7/d28d3f47-b0c1-4fbb-bdab-a8b85a0388d0"
-					(reference "C?")
+					(reference "C306")
 					(unit 1)
 				)
@@
 		(on_board yes)
 		(dnp no)
-		(property "Reference" "U?"
-			(at 60.706 29.972 0)
+		(property "Reference" "U301"
+			(at 58.928 29.972 0)
 			(effects
 				(font
@@
 			(project "shopie-hw"
 				(path "/e9514a67-47f8-4b41-a728-bdf26e012bf7/d28d3f47-b0c1-4fbb-bdab-a8b85a0388d0"
-					(reference "U?")
+					(reference "U301")
 					(unit 1)
 				)
@@
 		(on_board yes)
 		(dnp no)
-		(property "Reference" "C?"
+		(property "Reference" "C305"
 			(at 160.528 41.402 0)
 			(effects
@@
 			(project "shopie-hw"
 				(path "/e9514a67-47f8-4b41-a728-bdf26e012bf7/d28d3f47-b0c1-4fbb-bdab-a8b85a0388d0"
-					(reference "C?")
+					(reference "C305")
 					(unit 1)
 				)

Commit message: Add custom ESC footprint
- Created through-hole pads for ESC mounting with 4mm diameter holes and copper rings on top and bottom layers
- Included pads for GND, 4 motor PWM signals, TX, and CURR monitoring
- Verified pad dimensions and alignment with ESC wire specifications
Parts:
- U5: footprint (none) -> ShopieLibrary:HAKRC_Blehli32_ESC40A
Connections:
- net +BATT: now also U5.5 (BATT-), U5.7 (GND); no longer U5. (M1P1)
- net ADC1_IN1: now also U5.13 (CURR); no longer U5. (M1P1)
- net TIM2_CH1: now also U5.8 (S1); no longer U5. (M1P1)
- net TIM3_CH1: now also U5.9 (S2); no longer U5. (M1P1)
- net TIM4_CH1: now also U5.10 (S3); no longer U5. (M1P1)
- net TIM5_CH1: now also U5.11 (S4); no longer U5. (M1P1)
- net USART3_RX: now also U5.12 (TX); no longer U5. (M1P1)
- net VCharger: now also U5.6 (BATT+); no longer U5. (M1P1)
Changed lines of the file:
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@@
 	(wire
 		(pts
+			(xy 60.96 109.22) (xy 58.42 109.22)
+		)
+		(stroke
+			(width 0)
+			(type default)
+		)
+	)
+	(wire
+		(pts
 			(xy 72.39 66.04) (xy 53.34 66.04)
 		)
@@
 	(wire
 		(pts
+			(xy 60.96 111.76) (xy 60.96 109.22)
+		)
+		(stroke
+			(width 0)
+			(type default)
+		)
+	)
+	(wire
+		(pts
 			(xy 176.53 31.75) (xy 182.88 31.75)
 		)
@@
 	(wire
 		(pts
-			(xy 198.12 39.37) (xy 200.66 39.37)
+			(xy 58.42 105.41) (xy 62.23 105.41)
 		)
 		(stroke
@@
 	(wire
 		(pts
-			(xy 182.88 40.64) (xy 182.88 34.29)
+			(xy 198.12 39.37) (xy 200.66 39.37)
 		)
 		(stroke
@@
 	(wire
 		(pts
-			(xy 104.14 48.26) (xy 107.95 48.26)
+			(xy 182.88 40.64) (xy 182.88 34.29)
 		)
 		(stroke
@@
 	(wire
 		(pts
-			(xy 58.42 109.22) (xy 62.23 109.22)
+			(xy 104.14 48.26) (xy 107.95 48.26)
 		)
 		(stroke
@@
 	(wire
 		(pts
-			(xy 58.42 105.41) (xy 60.96 105.41)
-		)
-		(stroke
-			(width 0)
-			(type default)
-		)
-	)
-	(wire
-		(pts
 			(xy 260.35 41.91) (xy 264.16 41.91)
 		)
@@
 	(symbol
 		(lib_id "power:GND")
-		(at 60.96 105.41 90)
+		(at 60.96 111.76 0)
 		(unit 1)
 		(exclude_from_sim no)
@@
 		(dnp no)
 		(property "Reference" "#PWR045"
-			(at 67.31 105.41 0)
+			(at 60.96 118.11 0)
 			(effects
 				(font
@@
 		)
 		(property "Value" "GND"
-			(at 65.278 103.378 0)
+			(at 62.992 116.078 0)
 			(effects
 				(font
@@
 		)
 		(property "Footprint" ""
-			(at 60.96 105.41 0)
+			(at 60.96 111.76 0)
 			(effects
 				(font
@@
 		)
 		(property "Datasheet" ""
-			(at 60.96 105.41 0)
+			(at 60.96 111.76 0)
 			(effects
 				(font
@@
 		)
 		(property "Description" "Power symbol creates a global label with name \"GND\" , ground"
-			(at 60.96 105.41 0)
+			(at 60.96 111.76 0)
 			(effects
 				(font
@@
 			)
 		)
-		(property "Footprint" ""
+		(property "Footprint" "ShopieLibrary:HAKRC_Blehli32_ESC40A"
 			(at 45.72 106.68 0)
 			(effects
@@
 			)
 		)
-		(pin ""
+		(pin "10"
 		)
-		(pin ""
+		(pin "8"
 		)
-		(pin ""
+		(pin "3"
 		)
-		(pin ""
+		(pin "5"
 		)
 		(pin ""
 		)
-		(pin ""
+		(pin "3"
 		)
-		(pin ""
+		(pin "7"
 		)
-		(pin ""
+		(pin "4"
 		)
-		(pin ""
+		(pin "1"
 		)
-		(pin ""
+		(pin "11"
 		)
-		(pin ""
+		(pin "2"
 		)
-		(pin ""
+		(pin "12"
 		)
-		(pin ""
+		(pin "1"
 		)
-		(pin ""
+		(pin "9"
 		)
-		(pin ""
+		(pin "2"
 		)
-		(pin ""
+		(pin "6"
 		)
-		(pin ""
+		(pin "4"
 		)
-		(pin ""
+		(pin "1"
 		)
-		(pin ""
+		(pin "4"
 		)
-		(pin ""
+		(pin "3"
 		)
-		(pin ""
+		(pin "2"
 		)
-		(pin ""
+		(pin "13"
 		)
 		(instances
@@
 	(symbol
 		(lib_id "power:LINE")
-		(at 62.23 109.22 270)
+		(at 62.23 105.41 270)
 		(unit 1)
 		(exclude_from_sim no)
@@
 		(dnp no)
 		(property "Reference" "#PWR044"
-			(at 58.42 109.22 0)
+			(at 58.42 105.41 0)
 			(effects
 				(font
@@
 		)
 		(property "Value" "V_USB_BAT"
-			(at 58.674 111.506 90)
+			(at 58.674 107.696 90)
 			(effects
 				(font
@@
 		)
 		(property "Footprint" ""
-			(at 62.23 109.22 0)
+			(at 62.23 105.41 0)
 			(effects
 				(font
@@
 		)
 		(property "Datasheet" ""
-			(at 62.23 109.22 0)
+			(at 62.23 105.41 0)
 			(effects
 				(font
@@
 		)
 		(property "Description" "Power symbol creates a global label with name \"LINE\""
-			(at 62.23 109.22 0)
+			(at 62.23 105.41 0)
 			(effects
 				(font

Commit message: added/updated key components with symbols, footprints, and details
- Crystal Oscillator:
  • Replaced unavailable X49SM8MSD2SC (8MHz HC-49S-SMD) with X322512MSB4SI (12MHz, SMD3225-4P)
  • Added 22pF capacitors (CC0603JRNPO9BN220) to crystal OSC_IN and OSC_OUT, grounded both

- Power Switches:
  • Evaluated and replaced unavailable ST-0-102-C03-N003-RS with 2MS1T1B1M2QES toggle switch (SPDT, 2A@250VAC, 3A@28VDC)

- BOOT0 Slide Switch:
  • Added BOOT0 slide switch (50mA DPDT SMD vertical)
  • Connected 10kΩ pull-down resistor between switch output and GND
  • Enables manual BOOT0 control for programming mode

- ST-LINK Header:
  • Selected 1x5P 2.54mm THT header for SWD (SWCLK, SWDIO, GND, 3.3V, SWO)
  • SWO enabled via STM32CubeIDE “Trace Asynchronous SW” debug mode

-  JST-XH Battery Balance Connector:
  • Matched HRB 4S LiPo JST-XH (5 black + 1 red wire) to BMS cell input pins
  • To be paired with JST-XH 6-pin male connector on PCB

-  Barrel Jack:
  • Added Symbol for barrel Jack

All components(Caps, Resistors, etc..) added with valid footprints.
Parts:
- C18: footprint (none) -> ShopieLibrary:CL21B105KBFNNNE
- C301, C302, C303, C304, C305, C306, C307, C308: footprint (none) -> ShopieLibrary:CL21B104KBCNNNC
- R301, R302, R303, R8, R9: footprint (none) -> ShopieLibrary:RC0603FR-074K7L
- R5: value 0R5 -> 00R5; footprint (none) -> ShopieLibrary:WSLP3921L5000FEA
Changed lines of the file:
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@@
 			)
 		)
-		(property "Footprint" ""
+		(property "Footprint" "ShopieLibrary:RC0603FR-074K7L"
 			(at 207.01 85.09 0)
 			(effects
@@
 			)
 		)
-		(property "Datasheet" "~"
+		(property "Datasheet" "https://lcsc.com/datasheet/lcsc_datasheet_2506161100_YAGEO-RC0603FR-074K7L_C99782.pdf"
 			(at 207.01 85.09 0)
 			(effects
@@
 			)
 		)
-		(property "Description" "Resistor, small symbol"
+		(property "Description" "RC0603FR-074K7L"
 			(at 207.01 85.09 0)
 			(effects
@@
 			)
 		)
-		(property "Footprint" ""
+		(property "Footprint" "ShopieLibrary:CL21B104KBCNNNC"
 			(at 261.3152 52.07 0)
 			(effects
@@
 			)
 		)
-		(property "Datasheet" "~"
+		(property "Datasheet" "https://lcsc.com/datasheet/lcsc_datasheet_2304140030_Samsung-Electro-Mechanics-CL21B104KBCNNNC_C1711.pdf"
 			(at 260.35 48.26 0)
 			(effects
@@
 			)
 		)
-		(property "Footprint" ""
+		(property "Footprint" "ShopieLibrary:CL21B104KBCNNNC"
 			(at 35.8648 24.13 0)
 			(effects
@@
 			)
 		)
-		(property "Datasheet" "~"
+		(property "Datasheet" "https://lcsc.com/datasheet/lcsc_datasheet_2304140030_Samsung-Electro-Mechanics-CL21B104KBCNNNC_C1711.pdf"
 			(at 36.83 27.94 0)
 			(effects
@@
 		(dnp no)
 		(property "Reference" "R302"
-			(at 199.39 49.53 0)
+			(at 200.66 49.022 0)
 			(effects
 				(font
@@
 			)
 		)
-		(property "Footprint" ""
+		(property "Footprint" "ShopieLibrary:RC0603FR-074K7L"
 			(at 196.85 52.07 0)
 			(effects
@@
 			)
 		)
-		(property "Datasheet" "~"
+		(property "Datasheet" "https://lcsc.com/datasheet/lcsc_datasheet_2506161100_YAGEO-RC0603FR-074K7L_C99782.pdf"
 			(at 196.85 52.07 0)
 			(effects
@@
 			)
 		)
-		(property "Description" "Resistor, small symbol"
+		(property "Description" "RC0603FR-074K7L"
 			(at 196.85 52.07 0)
 			(effects
@@
 		(dnp no)
 		(property "Reference" "R301"
-			(at 190.5 50.8 0)
+			(at 189.23 50.546 0)
 			(effects
 				(font
@@
 			)
 		)
-		(property "Footprint" ""
+		(property "Footprint" "ShopieLibrary:RC0603FR-074K7L"
 			(at 194.31 52.07 0)
 			(effects
@@
 			)
 		)
-		(property "Datasheet" "~"
+		(property "Datasheet" "https://lcsc.com/datasheet/lcsc_datasheet_2506161100_YAGEO-RC0603FR-074K7L_C99782.pdf"
 			(at 194.31 52.07 0)
 			(effects
@@
 			)
 		)
-		(property "Description" "Resistor, small symbol"
+		(property "Description" "RC0603FR-074K7L"
 			(at 194.31 52.07 0)
 			(effects
@@
 			)
 		)
-		(property "Footprint" ""
+		(property "Footprint" "ShopieLibrary:CL21B104KBCNNNC"
 			(at 71.4248 52.07 0)
 			(effects
@@
 			)
 		)
-		(property "Datasheet" "~"
+		(property "Datasheet" "https://lcsc.com/datasheet/lcsc_datasheet_2304140030_Samsung-Electro-Mechanics-CL21B104KBCNNNC_C1711.pdf"
 			(at 72.39 55.88 0)
 			(effects
@@
 			)
 		)
-		(property "Footprint" ""
+		(property "Footprint" "ShopieLibrary:CL21B105KBFNNNE"
 			(at 265.1252 95.25 0)
 			(effects
@@
 			)
 		)
-		(property "Datasheet" "~"
+		(property "Datasheet" "https://lcsc.com/datasheet/lcsc_datasheet_2304140030_Samsung-Electro-Mechanics-CL21B105KBFNNNE_C28323.pdf"
 			(at 264.16 91.44 0)
 			(effects
@@
 			)
 		)
-		(property "Value" "0R5"
+		(property "Value" "00R5"
 			(at 254 91.4399 0)
 			(effects
@@
 			)
 		)
-		(property "Footprint" ""
+		(property "Footprint" "ShopieLibrary:WSLP3921L5000FEA"
 			(at 251.46 90.17 0)
 			(effects
@@
 			)
 		)
-		(property "Datasheet" "~"
+		(property "Datasheet" "https://lcsc.com/datasheet/lcsc_datasheet_2410121736_Vishay-Intertech-WSLP3921L5000FEA_C413491.pdf"
 			(at 251.46 90.17 0)
 			(effects
@@
 			)
 		)
-		(property "Description" "Resistor, small symbol"
+		(property "Description" "WSLP3921L5000FEA"
 			(at 251.46 90.17 0)
 			(effects
@@
 			)
 		)
-		(property "Footprint" ""
+		(property "Footprint" "ShopieLibrary:CL21B104KBCNNNC"
 			(at 263.8552 34.29 0)
 			(effects
@@
 			)
 		)
-		(property "Datasheet" "~"
+		(property "Datasheet" "https://lcsc.com/datasheet/lcsc_datasheet_2304140030_Samsung-Electro-Mechanics-CL21B104KBCNNNC_C1711.pdf"
 			(at 262.89 30.48 0)
 			(effects
@@
 			)
 		)
-		(property "Footprint" ""
+		(property "Footprint" "ShopieLibrary:CL21B104KBCNNNC"
 			(at 70.8152 31.75 0)
 			(effects
@@
 			)
 		)
-		(property "Datasheet" "~"
+		(property "Datasheet" "https://lcsc.com/datasheet/lcsc_datasheet_2304140030_Samsung-Electro-Mechanics-CL21B104KBCNNNC_C1711.pdf"
 			(at 69.85 27.94 0)
 			(effects
@@
 			)
 		)
-		(property "Footprint" ""
+		(property "Footprint" "ShopieLibrary:CL21B104KBCNNNC"
 			(at 150.8252 46.99 0)
 			(effects
@@
 			)
 		)
-		(property "Datasheet" "~"
+		(property "Datasheet" "https://lcsc.com/datasheet/lcsc_datasheet_2304140030_Samsung-Electro-Mechanics-CL21B104KBCNNNC_C1711.pdf"
 			(at 149.86 43.18 0)
 			(effects
@@
 		(dnp no)
 		(property "Reference" "R303"
-			(at 204.47 53.34 0)
+			(at 206.248 53.34 0)
 			(effects
 				(font
@@
 			)
 		)
-		(property "Footprint" ""
+		(property "Footprint" "ShopieLibrary:RC0603FR-074K7L"
 			(at 200.66 52.07 0)
 			(effects
@@
 			)
 		)
-		(property "Datasheet" "~"
+		(property "Datasheet" "https://lcsc.com/datasheet/lcsc_datasheet_2506161100_YAGEO-RC0603FR-074K7L_C99782.pdf"
 			(at 200.66 52.07 0)
 			(effects
@@
 			)
 		)
-		(property "Description" "Resistor, small symbol"
+		(property "Description" "RC0603FR-074K7L"
 			(at 200.66 52.07 0)
 			(effects
@@
 			)
 		)
-		(property "Footprint" ""
+		(property "Footprint" "ShopieLibrary:RC0603FR-074K7L"
 			(at 200.66 85.09 0)
 			(effects
@@
 			)
 		)
-		(property "Datasheet" "~"
+		(property "Datasheet" "https://lcsc.com/datasheet/lcsc_datasheet_2506161100_YAGEO-RC0603FR-074K7L_C99782.pdf"
 			(at 200.66 85.09 0)
 			(effects
@@
 			)
 		)
-		(property "Description" "Resistor, small symbol"
+		(property "Description" "RC0603FR-074K7L"
 			(at 200.66 85.09 0)
 			(effects
@@
 			)
 		)
-		(property "Footprint" ""
+		(property "Footprint" "ShopieLibrary:CL21B104KBCNNNC"
 			(at 177.4952 40.64 0)
 			(effects
@@
 			)
 		)
-		(property "Datasheet" "~"
+		(property "Datasheet" "https://lcsc.com/datasheet/lcsc_datasheet_2304140030_Samsung-Electro-Mechanics-CL21B104KBCNNNC_C1711.pdf"
 			(at 176.53 36.83 0)
 			(effects
@@
 			)
 		)
-		(property "Footprint" ""
+		(property "Footprint" "ShopieLibrary:CL21B104KBCNNNC"
 			(at 159.7152 46.99 0)
 			(effects
@@
 			)
 		)
-		(property "Datasheet" "~"
+		(property "Datasheet" "https://lcsc.com/datasheet/lcsc_datasheet_2304140030_Samsung-Electro-Mechanics-CL21B104KBCNNNC_C1711.pdf"
 			(at 158.75 43.18 0)
 			(effects
